Commit message: feat: Update robot URDF dimensions and camera pose, adjust Ackermann wheelbase, configure Nav2 with SmacPlannerHybrid, and refresh example trajectory data.

File: src/robot_bringup/description/robot.urdf (robot description, URDF)
Before this commit: robot robot_name, 3 links, 2 joints
Links:
- link base_link: geometry visual box size=1.0 1.0 0.5
Joints:
- joint base_to_camera: origin xyz=0.1 0 0.1 rpy=0 0 0 -> xyz=0.45 0 1.5 rpy=0 0 0

Commit message: feat: Update ackermann_msgs, pointcloud_to_laserscan, and robot_bringup packages, and remove perception_vslam bridge.

File: src/robot_bringup/description/robot.urdf (robot description, URDF)
Before this commit: robot robot_name, 3 links, 2 joints
Links:
- added link base_footprint
- added link front_left_steering_link; visual cylinder length=0.05 radius=0.05
- added link front_left_wheel; visual cylinder length=0.1 radius=0.15
- added link front_right_steering_link; visual cylinder length=0.05 radius=0.05
- added link front_right_wheel; visual cylinder length=0.1 radius=0.15
- added link rear_left_wheel; visual cylinder length=0.1 radius=0.15
- added link rear_right_wheel; visual cylinder length=0.1 radius=0.15
- link base_link: geometry collision box size=1.0 0.6 0.3; visual box size=1.0 0.6 0.3
- link lidar_link: geometry visual cylinder length=0.05 radius=0.05
Joints:
- added joint base_joint: type fixed, parent base_link, child base_footprint, origin xyz=0 0 0 rpy=0 0 0
- added joint front_left_steering_joint: type revolute, parent base_link, child front_left_steering_link, origin xyz=0.425 0.35 0.15 rpy=0 0 0, axis 0 0 1, limit lower=-0.5 upper=0.5 effort=100 velocity=1.0
- added joint front_left_wheel_joint: type continuous, parent front_left_steering_link, child front_left_wheel, origin xyz=0 0 0 rpy=0 0 0, axis 0 1 0
- added joint front_right_steering_joint: type revolute, parent base_link, child front_right_steering_link, origin xyz=0.425 -0.35 0.15 rpy=0 0 0, axis 0 0 1, limit lower=-0.5 upper=0.5 effort=100 velocity=1.0
- added joint front_right_wheel_joint: type continuous, parent front_right_steering_link, child front_right_wheel, origin xyz=0 0 0 rpy=0 0 0, axis 0 1 0
- added joint rear_left_wheel_joint: type continuous, parent base_link, child rear_left_wheel, origin xyz=-0.425 0.35 0.15 rpy=0 0 0, axis 0 1 0
- added joint rear_right_wheel_joint: type continuous, parent base_link, child rear_right_wheel, origin xyz=-0.425 -0.35 0.15 rpy=0 0 0, axis 0 1 0
- joint base_to_camera: origin xyz=0.45 0 1.5 rpy=0 0 0 -> xyz=0.45 0 0.325 rpy=0 0 0
- joint base_to_lidar: origin xyz=0 0 0.2 rpy=0 0 0 -> xyz=0.2 0 0.325 rpy=0 0 0

Commit message: feat: Update VSLAM and mapping configurations, refine teleop steering, and add Nav2 activation script.

File: src/robot_bringup/description/robot.urdf (robot description, URDF)
Before this commit: robot ackermann_robot, 10 links, 9 joints
Links:
- link base_link: geometry collision box size=1.0 0.6 0.3; visual box size=0.02 0.1 0.05
- link camera_link: geometry visual box size=0.05 0.15 0.05; visual cylinder length=0.055 radius=0.02
- link front_left_wheel: geometry visual cylinder length=0.1 radius=0.15; visual cylinder length=0.105 radius=0.08
- link front_right_wheel: geometry visual cylinder length=0.1 radius=0.15; visual cylinder length=0.105 radius=0.08
- link rear_left_wheel: geometry visual cylinder length=0.1 radius=0.15; visual cylinder length=0.105 radius=0.08
- link rear_right_wheel: geometry visual cylinder length=0.1 radius=0.15; visual cylinder length=0.105 radius=0.08

Commit message: feat: Refine firmware safety, steering control, and update ROS2 navigation and perception configurations

File: src/robot_bringup/description/robot.urdf (robot description, URDF)
Before this commit: robot ackermann_robot, 10 links, 9 joints
Links:
- removed link lidar_link
- link base_link: geometry collision box size=0.8 1.16 0.3; visual box size=0.02 0.1 0.05
Joints:
- removed joint base_to_lidar
- joint base_to_camera: origin xyz=0.45 0 0.325 rpy=0 0 0 -> xyz=0.45 0 0.325 rpy=0 0.175 0
- joint front_left_steering_joint: origin xyz=0.425 0.35 0.15 rpy=0 0 0 -> xyz=0.3 0.58 0.15 rpy=0 0 0
- joint front_right_steering_joint: origin xyz=0.425 -0.35 0.15 rpy=0 0 0 -> xyz=0.3 -0.58 0.15 rpy=0 0 0
- joint rear_left_wheel_joint: origin xyz=-0.425 0.35 0.15 rpy=0 0 0 -> xyz=-0.3 0.58 0.15 rpy=0 0 0
- joint rear_right_wheel_joint: origin xyz=-0.425 -0.35 0.15 rpy=0 0 0 -> xyz=-0.3 -0.58 0.15 rpy=0 0 0

Commit message: feat: Implement firmware for new steering, drive, safety, and HAL components, and update ROS configs for reduced steering angle.

File: src/robot_bringup/description/robot.urdf (robot description, URDF)
Before this commit: robot ackermann_robot, 9 links, 8 joints
Links:
- added link imu_link; visual box size=0.02 0.02 0.005
Joints:
- added joint base_to_imu: type fixed, parent base_link, child imu_link, origin xyz=0 0 0.29 rpy=0 0 0
- joint front_left_steering_joint: limit lower=-0.5 upper=0.5 effort=100 velocity=1.0 -> lower=-0.1745 upper=0.1745 effort=100 velocity=1.0
- joint front_right_steering_joint: limit lower=-0.5 upper=0.5 effort=100 velocity=1.0 -> lower=-0.1745 upper=0.1745 effort=100 velocity=1.0

Commit message: feat: Add sensor fusion package with adaptive fusion logic and status displays, and adjust steering limits and firmware update rates.

File: src/robot_bringup/description/robot.urdf (robot description, URDF)
Before this commit: robot ackermann_robot, 10 links, 9 joints
Links:
- added link camera_accel_frame
- added link camera_accel_optical_frame
- added link camera_color_frame
- added link camera_color_optical_frame
- added link camera_depth_frame
- added link camera_depth_optical_frame
- added link camera_gyro_frame
- added link camera_gyro_optical_frame
- added link camera_ir_frame
- added link camera_ir_optical_frame
Joints:
- added joint camera_accel_to_optical: type fixed, parent camera_accel_frame, child camera_accel_optical_frame, origin xyz=0 0 0 rpy=-1.5707963 0 -1.5707963
- added joint camera_color_to_optical: type fixed, parent camera_color_frame, child camera_color_optical_frame, origin xyz=0 0 0 rpy=-1.5707963 0 -1.5707963
- added joint camera_depth_to_optical: type fixed, parent camera_depth_frame, child camera_depth_optical_frame, origin xyz=0 0 0 rpy=-1.5707963 0 -1.5707963
- added joint camera_gyro_to_optical: type fixed, parent camera_gyro_frame, child camera_gyro_optical_frame, origin xyz=0 0 0 rpy=-1.5707963 0 -1.5707963
- added joint camera_ir_to_optical: type fixed, parent camera_ir_frame, child camera_ir_optical_frame, origin xyz=0 0 0 rpy=-1.5707963 0 -1.5707963
- added joint camera_to_accel: type fixed, parent camera_link, child camera_accel_frame, origin xyz=0 0 0 rpy=0 0 0
- added joint camera_to_color: type fixed, parent camera_link, child camera_color_frame, origin xyz=0 0 0 rpy=0 0 0
- added joint camera_to_depth: type fixed, parent camera_link, child camera_depth_frame, origin xyz=0 0 0 rpy=0 0 0
- added joint camera_to_gyro: type fixed, parent camera_link, child camera_gyro_frame, origin xyz=0 0 0 rpy=0 0 0
- added joint camera_to_ir: type fixed, parent camera_link, child camera_ir_frame, origin xyz=0 0 0 rpy=0 0 0
- joint base_to_camera: origin xyz=0.45 0 0.325 rpy=0 0.175 0 -> xyz=0.45 0 0.325 rpy=0 0 0

Commit message: feat: Implement micro-ROS time synchronization, update robot URDF dimensions and sensor placements, adjust pointcloud-to-laserscan height limits, and revise navigation stack documentation with new nodes

File: src/robot_bringup/description/robot.urdf (robot description, URDF)
Before this commit: robot ackermann_robot, 20 links, 19 joints
Links:
- link base_link: geometry collision box size=0.8 1.16 0.57; visual box size=0.02 0.1 0.05
Joints:
- joint base_to_camera: origin xyz=0.45 0 0.325 rpy=0 0 0 -> xyz=0.45 0 0.57 rpy=0 0 0
- joint base_to_imu: origin xyz=0 0 0.29 rpy=0 0 0 -> xyz=0 0 0.58 rpy=0 0 0
